Commit message: Tuning, added writeout of poses to assets writer

File: cartographer_ros/urdf/sep8.urdf (robot description, URDF)
Before this commit: robot mvsec, 3 links, 2 joints
Links:
- added link odom; visual cylinder length=0.07 radius=0.05
Joints:
- added joint odom_joint: type fixed, parent base_link, child odom, origin xyz=0 0 0 rpy=0 0 0
